File: kicad/RGB/RGB.sch (KiCad schematic (older format))
At the start: 15 parts, among them SW1 SW_Push, U1 ATmega16A-AU, Y1 16Mhz

Commit message: Replaced ATMega16-16AU by ATMega16-16PU
Parts:
- removed U1: ATmega16A-AU, Package_QFP:TQFP-44_10x10mm_P0.8mm, symbol MCU_Microchip_ATmega:ATmega16A-AU
- added U2: ATmega16-16PU, Package_DIP:DIP-40_W15.24mm, symbol MCU_Microchip_ATmega:ATmega16-16PU
Connections:
- net B: now also U2.19 (PD5)
- net BLUE: now also U2.8 (PB7)
- net G: now also U2.18 (PD4)
- net GND: now also U2.11 (GND), U2.31 (GND)
- net GREEN: now also U2.7 (PB6)
- net OSC1: now also U2.13 (XTAL1)
- net OSC2: now also U2.12 (XTAL2)
- net R: now also U2.4 (PB3)
- net RED: now also U2.6 (PB5)
- net RESET: now also U2.9 (~RESET)
- net VCC: now also U2.10 (VCC), U2.30 (AVCC)
- net at D2.2 (A): now also U2.29 (PC7)
Other:
- moved on the sheet: C1, C2, Y1
Changed lines of the file:
@@
 Comment4 ""
 $EndDescr
-$Comp
-L MCU_Microchip_ATmega:ATmega16A-AU U1
-U 1 1 60ABB650
-P 4550 3500
-F 0 "U1" H 4550 1411 50  0000 C CNN
-F 1 "ATmega16A-AU" H 4550 1320 50  0000 C CNN
-F 2 "Package_QFP:TQFP-44_10x10mm_P0.8mm" H 4550 3500 50  0001 C CIN
-F 3 "http://ww1.microchip.com/downloads/en/DeviceDoc/Atmel-8154-8-bit-AVR-ATmega16A_Datasheet.pdf" H 4550 3500 50  0001 C CNN
-	1    4550 3500
-	1    0    0    -1
-$EndComp
 Text GLabel 3400 1800 0    50   Input ~ 0
 RESET
-Wire Wire Line
-	3400 1800 3950 1800
 Text GLabel 7000 1450 0    50   Input ~ 0
 RESET
@@
 Text GLabel 3400 2200 0    50   Input ~ 0
 OSC2
-Wire Wire Line
-	3400 2200 3950 2200
-Wire Wire Line
-	3400 2000 3950 2000
 $Comp
 L Device:Crystal Y1
 U 1 1 60AC6B76
-P 2100 3450
-F 0 "Y1" H 2100 3718 50  0000 C CNN
-F 1 "16Mhz" H 2100 3627 50  0000 C CNN
-F 2 "" H 2100 3450 50  0001 C CNN
-F 3 "~" H 2100 3450 50  0001 C CNN
-	1    2100 3450
-	1    0    0    -1
-$EndComp
-Text GLabel 1400 3450 0    50   Input ~ 0
+P 1600 1100
+F 0 "Y1" H 1600 1368 50  0000 C CNN
+F 1 "16Mhz" H 1600 1277 50  0000 C CNN
+F 2 "" H 1600 1100 50  0001 C CNN
+F 3 "~" H 1600 1100 50  0001 C CNN
+	1    1600 1100
+	1    0    0    -1
+$EndComp
+Text GLabel 900  1100 0    50   Input ~ 0
 OSC1
-Text GLabel 2700 3450 2    50   Input ~ 0
+Text GLabel 2200 1100 2    50   Input ~ 0
 OSC2
 $Comp
 L Device:C C1
 U 1 1 60AC7819
-P 1650 3900
-F 0 "C1" H 1765 3946 50  0000 L CNN
-F 1 "22pF" H 1765 3855 50  0000 L CNN
-F 2 "" H 1688 3750 50  0001 C CNN
-F 3 "~" H 1650 3900 50  0001 C CNN
-	1    1650 3900
+P 1150 1550
+F 0 "C1" H 1265 1596 50  0000 L CNN
+F 1 "22pF" H 1265 1505 50  0000 L CNN
+F 2 "" H 1188 1400 50  0001 C CNN
+F 3 "~" H 1150 1550 50  0001 C CNN
+	1    1150 1550
 	1    0    0    -1
 $EndComp
@@
 L Device:C C2
 U 1 1 60AC7BEE
-P 2550 3900
-F 0 "C2" H 2665 3946 50  0000 L CNN
-F 1 "22pF" H 2665 3855 50  0000 L CNN
-F 2 "" H 2588 3750 50  0001 C CNN
-F 3 "~" H 2550 3900 50  0001 C CNN
-	1    2550 3900
+P 2050 1550
+F 0 "C2" H 2165 1596 50  0000 L CNN
+F 1 "22pF" H 2165 1505 50  0000 L CNN
+F 2 "" H 2088 1400 50  0001 C CNN
+F 3 "~" H 2050 1550 50  0001 C CNN
+	1    2050 1550
 	1    0    0    -1
 $EndComp
@@
 L power:GND #PWR03
 U 1 1 60AC8097
-P 1650 4350
-F 0 "#PWR03" H 1650 4100 50  0001 C CNN
-F 1 "GND" H 1655 4177 50  0000 C CNN
-F 2 "" H 1650 4350 50  0001 C CNN
-F 3 "" H 1650 4350 50  0001 C CNN
-	1    1650 4350
+P 1150 2000
+F 0 "#PWR03" H 1150 1750 50  0001 C CNN
+F 1 "GND" H 1155 1827 50  0000 C CNN
+F 2 "" H 1150 2000 50  0001 C CNN
+F 3 "" H 1150 2000 50  0001 C CNN
+	1    1150 2000
 	1    0    0    -1
 $EndComp
@@
 L power:GND #PWR04
 U 1 1 60AC85EB
-P 2550 4350
-F 0 "#PWR04" H 2550 4100 50  0001 C CNN
-F 1 "GND" H 2555 4177 50  0000 C CNN
-F 2 "" H 2550 4350 50  0001 C CNN
-F 3 "" H 2550 4350 50  0001 C CNN
-	1    2550 4350
-	1    0    0    -1
-$EndComp
-Wire Wire Line
-	1400 3450 1650 3450
-Wire Wire Line
-	2250 3450 2550 3450
-Wire Wire Line
-	1650 3750 1650 3450
-Connection ~ 1650 3450
-Wire Wire Line
-	1650 3450 1950 3450
-Wire Wire Line
-	2550 3750 2550 3450
-Connection ~ 2550 3450
-Wire Wire Line
-	2550 3450 2700 3450
-Wire Wire Line
-	1650 4050 1650 4350
-Wire Wire Line
-	2550 4050 2550 4350
+P 2050 2000
+F 0 "#PWR04" H 2050 1750 50  0001 C CNN
+F 1 "GND" H 2055 1827 50  0000 C CNN
+F 2 "" H 2050 2000 50  0001 C CNN
+F 3 "" H 2050 2000 50  0001 C CNN
+	1    2050 2000
+	1    0    0    -1
+$EndComp
+Wire Wire Line
+	900  1100 1150 1100
+Wire Wire Line
+	1750 1100 2050 1100
+Wire Wire Line
+	1150 1400 1150 1100
+Connection ~ 1150 1100
+Wire Wire Line
+	1150 1100 1450 1100
+Wire Wire Line
+	2050 1400 2050 1100
+Connection ~ 2050 1100
+Wire Wire Line
+	2050 1100 2200 1100
+Wire Wire Line
+	1150 1700 1150 2000
+Wire Wire Line
+	2050 1700 2050 2000
 $Comp
 L Device:R_POT RV1
@@
 $EndComp
 Wire Wire Line
+	7800 2700 8250 2700
+$Comp
+L power:VCC #PWR013
+U 1 1 60B0CA7B
+P 4600 1000
+F 0 "#PWR013" H 4600 850 50  0001 C CNN
+F 1 "VCC" H 4615 1173 50  0000 C CNN
+F 2 "" H 4600 1000 50  0001 C CNN
+F 3 "" H 4600 1000 50  0001 C CNN
+	1    4600 1000
+	1    0    0    -1
+$EndComp
+$Comp
+L power:PWR_FLAG #FLG01
+U 1 1 60B0EBDC
+P 4750 1150
+F 0 "#FLG01" H 4750 1225 50  0001 C CNN
+F 1 "PWR_FLAG" V 4750 1278 50  0000 L CNN
+F 2 "" H 4750 1150 50  0001 C CNN
+F 3 "~" H 4750 1150 50  0001 C CNN
+	1    4750 1150
+	0    1    1    0
+$EndComp
+$Comp
+L power:PWR_FLAG #FLG02
+U 1 1 60B1085B
+P 4700 5800
+F 0 "#FLG02" H 4700 5875 50  0001 C CNN
+F 1 "PWR_FLAG" V 4700 5928 50  0000 L CNN
+F 2 "" H 4700 5800 50  0001 C CNN
+F 3 "~" H 4700 5800 50  0001 C CNN
+	1    4700 5800
+	0    1    1    0
+$EndComp
+Wire Wire Line
+	4700 5800 4550 5800
+Wire Wire Line
+	4550 5800 4550 5850
+$Comp
+L Device:LED D2
+U 1 1 60B1F77D
+P 5450 4300
+F 0 "D2" H 5443 4045 50  0000 C CNN
+F 1 "RED" H 5443 4136 50  0000 C CNN
+F 2 "" H 5450 4300 50  0001 C CNN
+F 3 "~" H 5450 4300 50  0001 C CNN
+	1    5450 4300
+	-1   0    0    1
+$EndComp
+$Comp
+L Device:R R5
+U 1 1 60B223D3
+P 5850 4300
+F 0 "R5" V 5643 4300 50  0000 C CNN
+F 1 "200" V 5734 4300 50  0000 C CNN
+F 2 "" V 5780 4300 50  0001 C CNN
+F 3 "~" H 5850 4300 50  0001 C CNN
+	1    5850 4300
+	0    1    1    0
+$EndComp
+$Comp
+L power:GND #PWR014
+U 1 1 60B22910
+P 6150 4300
+F 0 "#PWR014" H 6150 4050 50  0001 C CNN
+F 1 "GND" V 6155 4172 50  0000 R CNN
+F 2 "" H 6150 4300 50  0001 C CNN
+F 3 "" H 6150 4300 50  0001 C CNN
+	1    6150 4300
+	0    -1   -1   0
+$EndComp
+Wire Wire Line
+	5600 4300 5700 4300
+Wire Wire Line
+	6000 4300 6150 4300
+$Comp
+L MCU_Microchip_ATmega:ATmega16-16PU U2
+U 1 1 60B2776C
+P 4550 3500
+F 0 "U2" H 4550 1411 50  0000 C CNN
+F 1 "ATmega16-16PU" H 4550 1320 50  0000 C CNN
+F 2 "Package_DIP:DIP-40_W15.24mm" H 4550 3500 50  0001 C CIN
+F 3 "http://ww1.microchip.com/downloads/en/DeviceDoc/doc2466.pdf" H 4550 3500 50  0001 C CNN
+	1    4550 3500
+	1    0    0    -1
+$EndComp
+Wire Wire Line
+	3400 1800 3950 1800
+Wire Wire Line
+	3400 2000 3950 2000
+Wire Wire Line
+	3400 2200 3950 2200
+Wire Wire Line
+	4550 1500 4550 1000
+Wire Wire Line
+	4550 1000 4600 1000
+Wire Wire Line
+	4650 1500 4650 1150
+Wire Wire Line
+	4650 1000 4600 1000
+Connection ~ 4600 1000
+Wire Wire Line
+	4750 1150 4650 1150
+Connection ~ 4650 1150
+Wire Wire Line
+	4650 1150 4650 1000
+Wire Wire Line
+	5150 3000 5450 3000
+Wire Wire Line
+	5150 3200 5400 3200
+Wire Wire Line
+	5150 3300 5400 3300
+Wire Wire Line
+	5150 3400 5400 3400
+Wire Wire Line
+	5150 4300 5300 4300
+Wire Wire Line
+	5150 4900 5500 4900
+Wire Wire Line
+	5150 5000 5500 5000
+Wire Wire Line
 	4550 5500 4550 5800
+Connection ~ 4550 5800
 NoConn ~ 3950 2400
-NoConn ~ 5150 2100
-NoConn ~ 5150 2200
-NoConn ~ 5150 2300
-NoConn ~ 5150 2400
-NoConn ~ 5150 2500
 NoConn ~ 5150 2700
 NoConn ~ 5150 2800
@@
 NoConn ~ 5150 4100
 NoConn ~ 5150 4200
+NoConn ~ 5150 4500
+NoConn ~ 5150 4600
+NoConn ~ 5150 4700
 NoConn ~ 5150 4800
 NoConn ~ 5150 5100
 NoConn ~ 5150 5200
-Wire Wire Line
-	7800 2700 8250 2700
-$Comp
-L power:VCC #PWR013
-U 1 1 60B0CA7B
-P 4600 1000
-F 0 "#PWR013" H 4600 850 50  0001 C CNN
-F 1 "VCC" H 4615 1173 50  0000 C CNN
-F 2 "" H 4600 1000 50  0001 C CNN
-F 3 "" H 4600 1000 50  0001 C CNN
-	1    4600 1000
-	1    0    0    -1
-$EndComp
-Wire Wire Line
-	4600 1000 4550 1000
-Wire Wire Line
-	4550 1000 4550 1500
-Wire Wire Line
-	4600 1000 4650 1000
-Wire Wire Line
-	4650 1000 4650 1150
-Connection ~ 4600 1000
-$Comp
-L power:PWR_FLAG #FLG01
-U 1 1 60B0EBDC
-P 4750 1150
-F 0 "#FLG01" H 4750 1225 50  0001 C CNN
-F 1 "PWR_FLAG" V 4750 1278 50  0000 L CNN
-F 2 "" H 4750 1150 50  0001 C CNN
-F 3 "~" H 4750 1150 50  0001 C CNN
-	1    4750 1150
-	0    1    1    0
-$EndComp
-Wire Wire Line
-	4650 1150 4750 1150
-Connection ~ 4650 1150
-Wire Wire Line
-	4650 1150 4650 1500
-$Comp
-L power:PWR_FLAG #FLG02
-U 1 1 60B1085B
-P 4700 5800
-F 0 "#FLG02" H 4700 5875 50  0001 C CNN
-F 1 "PWR_FLAG" V 4700 5928 50  0000 L CNN
-F 2 "" H 4700 5800 50  0001 C CNN
-F 3 "~" H 4700 5800 50  0001 C CNN
-	1    4700 5800
-	0    1    1    0
-$EndComp
-Wire Wire Line
-	4700 5800 4550 5800
-Connection ~ 4550 5800
-Wire Wire Line
-	4550 5800 4550 5850
-Wire Wire Line
-	5150 5000 5500 5000
-Wire Wire Line
-	5150 4900 5500 4900
-Wire Wire Line
-	5150 3000 5450 3000
-NoConn ~ 5150 4500
-NoConn ~ 5150 4600
-NoConn ~ 5150 4700
-Wire Wire Line
-	5150 3200 5400 3200
-Wire Wire Line
-	5150 3300 5400 3300
-Wire Wire Line
-	5150 3400 5400 3400
 NoConn ~ 5150 1800
 NoConn ~ 5150 1900
 NoConn ~ 5150 2000
-$Comp
-L Device:LED D2
-U 1 1 60B1F77D
-P 5450 4300
-F 0 "D2" H 5443 4045 50  0000 C CNN
-F 1 "RED" H 5443 4136 50  0000 C CNN
-F 2 "" H 5450 4300 50  0001 C CNN
-F 3 "~" H 5450 4300 50  0001 C CNN
-	1    5450 4300
-	-1   0    0    1
-$EndComp
-Wire Wire Line
-	5150 4300 5300 4300
-$Comp
-L Device:R R5
-U 1 1 60B223D3
-P 5850 4300
-F 0 "R5" V 5643 4300 50  0000 C CNN
-F 1 "200" V 5734 4300 50  0000 C CNN
-F 2 "" V 5780 4300 50  0001 C CNN
-F 3 "~" H 5850 4300 50  0001 C CNN
-	1    5850 4300
-	0    1    1    0
-$EndComp
-$Comp
-L power:GND #PWR014
-U 1 1 60B22910
-P 6150 4300
-F 0 "#PWR014" H 6150 4050 50  0001 C CNN
-F 1 "GND" V 6155 4172 50  0000 R CNN
-F 2 "" H 6150 4300 50  0001 C CNN
-F 3 "" H 6150 4300 50  0001 C CNN
-	1    6150 4300
-	0    -1   -1   0
-$EndComp
-Wire Wire Line
-	5600 4300 5700 4300
-Wire Wire Line
-	6000 4300 6150 4300
+NoConn ~ 5150 2100
+NoConn ~ 5150 2200
+NoConn ~ 5150 2300
+NoConn ~ 5150 2400
+NoConn ~ 5150 2500
 $EndSCHEMATC

Commit message: Footprints added
Parts:
- C1, C2: footprint (none) -> Capacitor_THT:C_Disc_D3.0mm_W1.6mm_P2.50mm
- D1: footprint (none) -> LED_THT:LED_D5.0mm-4_RGB
- D2: footprint (none) -> LED_THT:LED_D3.0mm
- R1, R2, R3, R4, R5: footprint (none) -> Resistor_THT:R_Axial_DIN0309_L9.0mm_D3.2mm_P12.70mm_Horizontal
- RV1, RV2, RV3: footprint (none) -> Potentiometer_THT:Potentiometer_ACP_CA9-V10_Vertical
- SW1: footprint (none) -> Button_Switch_THT:Push_E-Switch_KS01Q01
- Y1: footprint (none) -> Crystal:Crystal_AT310_D3.0mm_L10.0mm_Horizontal
Changed lines of the file:
@@
 F 0 "SW1" H 7850 1615 50  0000 C CNN
 F 1 "SW_Push" H 7850 1706 50  0000 C CNN
-F 2 "" H 7850 2000 50  0001 C CNN
+F 2 "Button_Switch_THT:Push_E-Switch_KS01Q01" H 7850 2000 50  0001 C CNN
 F 3 "~" H 7850 2000 50  0001 C CNN
 	1    7850 1800
@@
 F 0 "R1" V 7593 1450 50  0000 C CNN
 F 1 "10K" V 7684 1450 50  0000 C CNN
-F 2 "" V 7730 1450 50  0001 C CNN
+F 2 "Resistor_THT:R_Axial_DIN0309_L9.0mm_D3.2mm_P12.70mm_Horizontal" V 7730 1450 50  0001 C CNN
 F 3 "~" H 7800 1450 50  0001 C CNN
 	1    7800 1450
@@
 F 0 "Y1" H 1600 1368 50  0000 C CNN
 F 1 "16Mhz" H 1600 1277 50  0000 C CNN
-F 2 "" H 1600 1100 50  0001 C CNN
+F 2 "Crystal:Crystal_AT310_D3.0mm_L10.0mm_Horizontal" H 1600 1100 50  0001 C CNN
 F 3 "~" H 1600 1100 50  0001 C CNN
 	1    1600 1100
@@
 F 0 "C1" H 1265 1596 50  0000 L CNN
 F 1 "22pF" H 1265 1505 50  0000 L CNN
-F 2 "" H 1188 1400 50  0001 C CNN
+F 2 "Capacitor_THT:C_Disc_D3.0mm_W1.6mm_P2.50mm" H 1188 1400 50  0001 C CNN
 F 3 "~" H 1150 1550 50  0001 C CNN
 	1    1150 1550
@@
 F 0 "C2" H 2165 1596 50  0000 L CNN
 F 1 "22pF" H 2165 1505 50  0000 L CNN
-F 2 "" H 2088 1400 50  0001 C CNN
+F 2 "Capacitor_THT:C_Disc_D3.0mm_W1.6mm_P2.50mm" H 2088 1400 50  0001 C CNN
 F 3 "~" H 2050 1550 50  0001 C CNN
 	1    2050 1550
@@
 F 0 "RV1" V 7443 2700 50  0000 C CNN
 F 1 "10K" V 7534 2700 50  0000 C CNN
-F 2 "" H 7650 2700 50  0001 C CNN
+F 2 "Potentiometer_THT:Potentiometer_ACP_CA9-V10_Vertical" H 7650 2700 50  0001 C CNN
 F 3 "~" H 7650 2700 50  0001 C CNN
 	1    7650 2700
@@
 F 0 "RV2" V 7443 3350 50  0000 C CNN
 F 1 "10K" V 7534 3350 50  0000 C CNN
-F 2 "" H 7650 3350 50  0001 C CNN
+F 2 "Potentiometer_THT:Potentiometer_ACP_CA9-V10_Vertical" H 7650 3350 50  0001 C CNN
 F 3 "~" H 7650 3350 50  0001 C CNN
 	1    7650 3350
@@
 F 0 "RV3" V 7443 4000 50  0000 C CNN
 F 1 "10K" V 7534 4000 50  0000 C CNN
-F 2 "" H 7650 4000 50  0001 C CNN
+F 2 "Potentiometer_THT:Potentiometer_ACP_CA9-V10_Vertical" H 7650 4000 50  0001 C CNN
 F 3 "~" H 7650 4000 50  0001 C CNN
 	1    7650 4000
@@
 F 0 "D1" H 8150 6097 50  0000 C CNN
 F 1 "LED_ARBG" H 8150 6006 50  0000 C CNN
-F 2 "" H 8150 5550 50  0001 C CNN
+F 2 "LED_THT:LED_D5.0mm-4_RGB" H 8150 5550 50  0001 C CNN
 F 3 "~" H 8150 5550 50  0001 C CNN
 	1    8150 5600
@@
 F 0 "R2" V 7250 5250 50  0000 C CNN
 F 1 "22" V 7250 5450 50  0000 C CNN
-F 2 "" V 7280 5400 50  0001 C CNN
+F 2 "Resistor_THT:R_Axial_DIN0309_L9.0mm_D3.2mm_P12.70mm_Horizontal" V 7280 5400 50  0001 C CNN
 F 3 "~" H 7350 5400 50  0001 C CNN
 	1    7350 5400
@@
 F 0 "R3" V 7250 5450 50  0000 C CNN
 F 1 "10" V 7250 5650 50  0000 C CNN
-F 2 "" V 7280 5600 50  0001 C CNN
+F 2 "Resistor_THT:R_Axial_DIN0309_L9.0mm_D3.2mm_P12.70mm_Horizontal" V 7280 5600 50  0001 C CNN
 F 3 "~" H 7350 5600 50  0001 C CNN
 	1    7350 5600
@@
 F 0 "R4" V 7250 5650 50  0000 C CNN
 F 1 "10" V 7250 5850 50  0000 C CNN
-F 2 "" V 7280 5800 50  0001 C CNN
+F 2 "Resistor_THT:R_Axial_DIN0309_L9.0mm_D3.2mm_P12.70mm_Horizontal" V 7280 5800 50  0001 C CNN
 F 3 "~" H 7350 5800 50  0001 C CNN
 	1    7350 5800
@@
 F 0 "D2" H 5443 4045 50  0000 C CNN
 F 1 "RED" H 5443 4136 50  0000 C CNN
-F 2 "" H 5450 4300 50  0001 C CNN
+F 2 "LED_THT:LED_D3.0mm" H 5450 4300 50  0001 C CNN
 F 3 "~" H 5450 4300 50  0001 C CNN
 	1    5450 4300
@@
 F 0 "R5" V 5643 4300 50  0000 C CNN
 F 1 "200" V 5734 4300 50  0000 C CNN
-F 2 "" V 5780 4300 50  0001 C CNN
+F 2 "Resistor_THT:R_Axial_DIN0309_L9.0mm_D3.2mm_P12.70mm_Horizontal" V 5780 4300 50  0001 C CNN
 F 3 "~" H 5850 4300 50  0001 C CNN
 	1    5850 4300
